File: pcb/leds.kicad_sch (KiCad schematic)
At the start: 36 parts

Commit message: feat(pcb): remove levelshifters, change to 3v3 vcc_io on tmc2209s, add rgb led to led driver, add R_ext value for led driver, add R_sense value for tmc2209s, add seperate dir signals for each tmc2209
Parts:
- removed LED35, LED36, LED37: (no value), lcsc:LED0603-R-RD_WHITE, symbol lcsc:0603Whitelight_C2290
- renumbered LED2 to LED1, LED11 to LED10, LED12 to LED11, LED13 to LED12, LED14 to LED13, LED15 to LED14, LED16 to LED15, LED17 to LED16, LED18 to LED17, LED19 to LED18, LED20 to LED19, LED3 to LED2, LED21 to LED20, LED22 to LED21, LED23 to LED22, LED24 to LED23, LED25 to LED24, LED26 to LED25, LED27 to LED26, LED28 to LED27, LED29 to LED28, LED30 to LED29, LED4 to LED3, LED31 to LED30, LED32 to LED31, LED33 to LED32, LED34 to LED33, LED5 to LED4, LED6 to LED5, LED7 to LED6, LED8 to LED7, LED9 to LED8, LED10 to LED9
