File: pcb/DrumTime.kicad_sch (KiCad schematic)
At the start: 45 parts, among them J1 EN, J2 Boot, J3 Debug, J4 LED_Conn, J5 LED_Conn, U1 ME6210A33PG, U2 ESP32-S3-WROOM-1-N8, U3 TJ-S1608SW6TDSLCCYRGB-A5, U4 IS31FL3236A-QFLS2-TR

Commit message: feat(pcb): layout motor drivers and route internally
Parts:
- removed H2: MountingHole, MountingHole:MountingHole_2.2mm_M2_Pad, symbol Mechanical:MountingHole_Pad
- J4, J5: footprint Connector_PinHeader_2.54mm:PinHeader_1x04_P2.54mm_Vertical -> Connector_JST:JST_XH_B4B-XH-AM_1x04_P2.50mm_Vertical
- renumbered H4 to H2, H5 to H4, H6 to H5
Other:
- moved on the sheet: H2

Commit message: feat(pcb): finish initial routing and layouting
Connections:
- net +5V: no longer U4.36 (SDB)
- net m0_dir: now also U2.5 (IO5); no longer U2.6 (IO6)
- net m0_hall: now also U2.4 (IO4); no longer U2.5 (IO5)
- net m0_step: now also U2.6 (IO6); no longer U2.4 (IO4)
- net m1_dir: now also U2.8 (IO15); no longer U2.9 (IO16)
- net m1_hall: now also U2.7 (IO7); no longer U2.8 (IO15)
- net m1_step: now also U2.9 (IO16); no longer U2.7 (IO7)
- net m2_dir: now also U2.17 (IO9); no longer U2.18 (IO10)
- net m2_hall: now also U2.12 (IO8); no longer U2.17 (IO9)
- net m2_step: now also U2.18 (IO10); no longer U2.12 (IO8)
- net m3_dir: now also U2.20 (IO12); no longer U2.21 (IO13)
- net m3_hall: now also U2.19 (IO11); no longer U2.20 (IO12)
- net m3_step: now also U2.21 (IO13); no longer U2.19 (IO11)
- net SDB: now reaches C11.1, C12.1, R9.2, U4.38 (VCC)
- net SDB: now also U4.36 (SDB)
